File: Base_Hardware/Base_Hardware.kicad_pcb (KiCad board)
At the start: 2 copper layers, 23 parts, among them J1 USB_B_Mini, J2 ISP, J3 NEO Out, SW1 SW_Push, U1 ATtiny85-20SU

Commit message: created tree outlines
Parts:
- moved D14 219.4 mm to (-55.3, 37.3)
- moved D13 208.5 mm to (-48.4, 38.4)
- moved D12 199.0 mm to (-41.3, 39.2)
- moved D10 193.4 mm to (-29.6, 39.7)
- moved D9 185.6 mm to (-23.3, 39.9)
- moved D11 175.3 mm to (-34.7, 39.4)
- moved U1 162.5 mm to (-16.2, 133.5)
- moved C1 154.6 mm to (-16.1, 117.7)
- moved D3 153.0 mm to (-30.4, 110.8)
- moved D6 153.0 mm to (-33.8, 110.8)
- moved J2 153.0 mm to (-31.8, 96.5)
- moved J3 153.0 mm to (-15.2, 92.7)
- moved SW1 153.0 mm to (-8.34, 94.3)
- moved D2 127.4 mm to (24.2, 93.3)
- moved R2 124.7 mm to (21.7, 117.5)
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Connections:
- net D+ renamed Net-(J1-Pad2)
- net D- renamed Net-(J1-Pad4)
- D1 pad 2: Net-(D1-Pad2) -> GND
- D10 pad 2: Net-(D1-Pad2) -> GND
- D11 pad 2: Net-(D1-Pad2) -> GND
- D12 pad 2: Net-(D1-Pad2) -> GND
- D13 pad 2: Net-(D1-Pad2) -> GND
- D14 pad 2: Net-(D1-Pad2) -> GND
- D2 pad 2: Net-(D1-Pad2) -> GND
- D4 pad 2: Net-(D1-Pad2) -> GND
- D5 pad 2: Net-(D1-Pad2) -> GND
- D7 pad 2: Net-(D1-Pad2) -> GND
- D8 pad 2: Net-(D1-Pad2) -> GND
- D9 pad 2: Net-(D1-Pad2) -> GND
- J1 pad 6: (no net) -> GND
Routing:
- added copper zone on B.Cu, net +5V
- added copper zone on F.Cu, net GND
Other:
- board outline added: 74.1 x 89 mm

Commit message: modified connecting slit
Parts:
- removed D14: SK6805, LED_SMD:LED_SK6805_PLCC4_2.4x2.7mm_P1.3mm
- D1, D10, D11, D12, D13, D2, D4, D5, D7, D8, D9: footprint LED_SMD:LED_SK6805_PLCC4_2.4x2.7mm_P1.3mm -> ProjectLibrary:SK6805-EC
- moved U1 176.7 mm to (160.0, 120.7)
- moved J2 168.6 mm to (136.1, 111.5)
- moved SW1 167.9 mm to (158.8, 110.5)
- moved J3 152.4 mm to (137.2, 94.0), turned to 270 degrees
- moved D1 149.5 mm to (175.5, 124.9)
- moved D13 106.2 mm to (48.3, 82.1)
- moved D12 97.2 mm to (44.4, 85.0)
- moved D10 91.2 mm to (52.6, 79.1)
- moved D9 83.0 mm to (53.2, 72.2)
- moved D11 75.3 mm to (24.9, 85.4)
- moved C1 64.0 mm to (40.2, 87.3)
- moved D3 59.2 mm to (24.2, 87.7)
- moved D6 59.2 mm to (20.8, 87.7)
- moved J1 52.6 mm to (122.2, 116.8)
- moved R2 42.4 mm to (48.1, 84.3)
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Connections:
- D13 pad 1: Net-(D13-Pad1) -> DOut'
Other:
- board size 74.1 x 89 mm -> 74.1 x 91.2 mm

Commit message: Placed high-level components and traces
Parts:
- J3: footprint Connector_PinSocket_2.54mm:PinSocket_1x03_P2.54mm_Horizontal -> Connector_PinSocket_2.54mm:PinSocket_1x03_P2.54mm_Vertical
- moved D6 137.4 mm to (155.6, 114.6), turned to 180 degrees
- moved D3 114.4 mm to (132.2, 125.2)
- moved C1 111.4 mm to (149.3, 110.0), turned to 180 degrees
- moved R3 107.6 mm to (151.8, 114.6)
- moved R2 97.0 mm to (136.0, 125.2), turned to 180 degrees
- moved U1 15.9 mm to (153.8, 106.0), turned to 180 degrees
- moved SW1 10.1 mm to (153.5, 119.1)
- moved J2 8.41 mm to (132.1, 104.1)
- moved J1 6.21 mm to (117.5, 121.0)
- moved J3 5.24 mm to (138.4, 88.9), turned to 0 degrees
Routing:
- net RST: track 0.00 -> 28.1 mm
- net Push: track 0.00 -> 26.4 mm
- net GND: track 0.00 -> 26.2 mm, vias 0 -> 7
- net MISO: track 0.00 -> 24.3 mm
- net SCK: track 0.00 -> 19.2 mm
- net MOSI: track 0.00 -> 16.6 mm
- net +5V: track 0.00 -> 12.4 mm, vias 0 -> 1
- net Net-(D6-Pad2): track 0.00 -> 2.03 mm
- net Net-(D3-Pad2): track 0.00 -> 2.03 mm
- added copper zone on F.Cu, net +5V
- added copper zone on B.Cu, net GND
- removed copper zone on B.Cu, net +5V
- removed copper zone on F.Cu, net GND

Commit message: Finished layout
Parts:
- D10, D12, D13, D2, D5, D8: moved to B.Cu
- moved D2 134.8 mm to (176.0, 124.9), turned to 270 degrees
- moved R1 132.3 mm to (170.6, 124.5), turned to 180 degrees
- moved D4 127.3 mm to (167.2, 94.4), turned to 180 degrees
- moved D8 120.3 mm to (159.5, 67.8), turned to 270 degrees
- moved D7 116.0 mm to (159.6, 67.8), turned to 180 degrees
- moved D5 116.0 mm to (167.2, 94.4), turned to 270 degrees
- moved D11 92.9 mm to (117.4, 94.5), turned to 90 degrees
- moved D13 73.6 mm to (108.2, 124.9)
- moved D12 73.6 mm to (117.4, 94.4), turned to 180 degrees
- moved D10 73.2 mm to (124.9, 67.8), turned to 180 degrees
- moved D9 71.8 mm to (124.9, 67.8), turned to 90 degrees
- moved D3 0.76 mm to (132.2, 124.5)
- moved R2 0.76 mm to (136.0, 124.5)
- moved D1 0.57 mm to (176.1, 124.9), turned to 180 degrees
Routing:
- net Net-(D8-Pad1): track 0.00 -> 72.5 mm, vias 0 -> 3
- net DOut': track 0.00 -> 65.3 mm, vias 0 -> 2
- net Net-(D12-Pad1): track 0.00 -> 50.5 mm, vias 0 -> 2
- net Net-(D2-Pad1): track 0.00 -> 47.5 mm, vias 0 -> 3
- net Net-(D5-Pad1): track 0.00 -> 41.4 mm, vias 0 -> 3
- net Net-(D10-Pad1): track 0.00 -> 41.3 mm, vias 0 -> 3
- net DOut: track 0.00 -> 30.4 mm, vias 0 -> 2
- net GND: track 26.2 -> 37.6 mm, vias 7 -> 13
- net +5V: track 12.4 -> 19.3 mm, vias 1 -> 7
- net Net-(D1-Pad3): track 0.00 -> 4.13 mm
- net Net-(D4-Pad1): track 0.00 -> 3.02 mm, vias 0 -> 1
- net Net-(D1-Pad1): track 0.00 -> 3.02 mm, vias 0 -> 1
- net Net-(D7-Pad1): track 0.00 -> 3.02 mm, vias 0 -> 1
- net Net-(D11-Pad1): track 0.00 -> 2.78 mm, vias 0 -> 1
- net Net-(D10-Pad3): track 0.00 -> 2.78 mm, vias 0 -> 1
Other:
- board text added: "Power"
- board text added: "R2"
